File: ParkingSystem/ParkingSystem.sch (KiCad schematic (older format))
At the start: 38 parts

Commit message: Add microfit footprints
Parts:
- J?: footprint (none) -> Connector_Molex:Molex_Micro-Fit_3.0_43045-0400_2x02_P3.00mm_Horizontal
- J?: footprint (none) -> Connector_Molex:Molex_Mega-Fit_76829-0108_2x04_P5.70mm_Vertical
Changed lines of the file:
@@
 F 0 "J?" H 2256 7075 50  0000 C CNN
 F 1 "0430450400" H 2256 6984 50  0000 C CNN
-F 2 "" H 2200 6650 50  0001 C CNN
+F 2 "Connector_Molex:Molex_Micro-Fit_3.0_43045-0400_2x02_P3.00mm_Horizontal" H 2200 6650 50  0001 C CNN
 F 3 "" H 2200 6650 50  0001 C CNN
 	1    2200 6650
@@
 F 0 "J?" H 2256 7625 50  0000 C CNN
 F 1 "0430450200" H 2256 7534 50  0000 C CNN
-F 2 "" H 2200 7350 50  0001 C CNN
+F 2 "Connector_Molex:Molex_Mega-Fit_76829-0108_2x04_P5.70mm_Vertical" H 2200 7350 50  0001 C CNN
 F 3 "" H 2200 7350 50  0001 C CNN
 	1    2200 7350

Commit message: Add Cortex Programming Header
Parts:
- removed J?: Conn_01x10_Male, symbol Connector:Conn_01x10_Male
- added J?: Conn_ARM_JTAG_SWD_10, Connector_PinHeader_1.27mm:PinHeader_2x05_P1.27mm_Vertical_SMD, symbol Connector:Conn_ARM_JTAG_SWD_10
- added R? (x2): 10K, Resistor_SMD:R_0603_1608Metric_Pad1.05x0.95mm_HandSolder, symbol Device:R_US
Connections:
- net labels added: SWDCLK, SWDIO, TDI, TDO
- wire segments 143 -> 161
Other:
- moved on the sheet: U?

Commit message: Add Crystal Oscillator
Parts:
- added C? (x2): 30p, Capacitor_SMD:C_0603_1608Metric_Pad1.05x0.95mm_HandSolder, symbol Device:C_Small
- added Y?: Crystal, symbol Device:Crystal
- D?: footprint (none) -> LED_SMD:LED_0603_1608Metric_Pad1.05x0.95mm_HandSolder
Connections:
- wire segments 161 -> 174
Other:
- moved on the sheet: D?, R?
Changed lines of the file:
@@
 L Device:LED D?
 U 1 1 5C67C377
-P 6150 1100
-F 0 "D?" V 6188 983 50  0000 R CNN
-F 1 "LED" V 6097 983 50  0000 R CNN
-F 2 "" H 6150 1100 50  0001 C CNN
-F 3 "~" H 6150 1100 50  0001 C CNN
-	1    6150 1100
+P 5850 1100
+F 0 "D?" V 5888 983 50  0000 R CNN
+F 1 "LED" V 5797 983 50  0000 R CNN
+F 2 "LED_SMD:LED_0603_1608Metric_Pad1.05x0.95mm_HandSolder" H 5850 1100 50  0001 C CNN
+F 3 "~" H 5850 1100 50  0001 C CNN
+	1    5850 1100
 	0    -1   -1   0
 $EndComp
@@
 L power:+3V3 #PWR0148
 U 1 1 5C67C58D
-P 6150 900
-F 0 "#PWR0148" H 6150 750 50  0001 C CNN
-F 1 "+3V3" H 6165 1073 50  0000 C CNN
-F 2 "" H 6150 900 50  0001 C CNN
-F 3 "" H 6150 900 50  0001 C CNN
-	1    6150 900
+P 5850 900
+F 0 "#PWR0148" H 5850 750 50  0001 C CNN
+F 1 "+3V3" H 5865 1073 50  0000 C CNN
+F 2 "" H 5850 900 50  0001 C CNN
+F 3 "" H 5850 900 50  0001 C CNN
+	1    5850 900
 	1    0    0    -1
 $EndComp
@@
 L power:GND #PWR0149
 U 1 1 5C67C622
-P 6150 1650
-F 0 "#PWR0149" H 6150 1400 50  0001 C CNN
-F 1 "GND" H 6155 1477 50  0000 C CNN
-F 2 "" H 6150 1650 50  0001 C CNN
-F 3 "" H 6150 1650 50  0001 C CNN
-	1    6150 1650
+P 5850 1650
+F 0 "#PWR0149" H 5850 1400 50  0001 C CNN
+F 1 "GND" H 5855 1477 50  0000 C CNN
+F 2 "" H 5850 1650 50  0001 C CNN
+F 3 "" H 5850 1650 50  0001 C CNN
+	1    5850 1650
 	1    0    0    -1
 $EndComp
@@
 L Device:R_US R?
 U 1 1 5C67C735
-P 6150 1450
-F 0 "R?" H 6218 1496 50  0000 L CNN
-F 1 "R_US" H 6218 1405 50  0000 L CNN
-F 2 "" V 6190 1440 50  0001 C CNN
-F 3 "~" H 6150 1450 50  0001 C CNN
-	1    6150 1450
-	1    0    0    -1
-$EndComp
-Wire Wire Line
-	6150 900  6150 950
-Wire Wire Line
-	6150 1250 6150 1300
-Wire Wire Line
-	6150 1650 6150 1600
+P 5850 1450
+F 0 "R?" H 5918 1496 50  0000 L CNN
+F 1 "R_US" H 5918 1405 50  0000 L CNN
+F 2 "" V 5890 1440 50  0001 C CNN
+F 3 "~" H 5850 1450 50  0001 C CNN
+	1    5850 1450
+	1    0    0    -1
+$EndComp
+Wire Wire Line
+	5850 900  5850 950
+Wire Wire Line
+	5850 1250 5850 1300
+Wire Wire Line
+	5850 1650 5850 1600
 Text Label 9350 2700 2    50   ~ 0
 BUZZER
@@
 L Device:R_US R?
 U 1 1 5C6B9C73
-P 7350 1550
-F 0 "R?" H 7282 1504 50  0000 R CNN
-F 1 "10K" H 7282 1595 50  0000 R CNN
-F 2 "Resistor_SMD:R_0603_1608Metric_Pad1.05x0.95mm_HandSolder" V 7390 1540 50  0001 C CNN
-F 3 "~" H 7350 1550 50  0001 C CNN
-	1    7350 1550
+P 6400 1550
+F 0 "R?" H 6332 1504 50  0000 R CNN
+F 1 "10K" H 6332 1595 50  0000 R CNN
+F 2 "Resistor_SMD:R_0603_1608Metric_Pad1.05x0.95mm_HandSolder" V 6440 1540 50  0001 C CNN
+F 3 "~" H 6400 1550 50  0001 C CNN
+	1    6400 1550
 	-1   0    0    1
 $EndComp
-Wire Wire Line
-	7700 1400 7350 1400
 $Comp
 L power:GND #PWR?
 U 1 1 5C6C098A
-P 7350 1750
-F 0 "#PWR?" H 7350 1500 50  0001 C CNN
-F 1 "GND" H 7355 1577 50  0000 C CNN
-F 2 "" H 7350 1750 50  0001 C CNN
-F 3 "" H 7350 1750 50  0001 C CNN
-	1    7350 1750
-	1    0    0    -1
-$EndComp
-Wire Wire Line
-	7350 1750 7350 1700
+P 6400 1750
+F 0 "#PWR?" H 6400 1500 50  0001 C CNN
+F 1 "GND" H 6405 1577 50  0000 C CNN
+F 2 "" H 6400 1750 50  0001 C CNN
+F 3 "" H 6400 1750 50  0001 C CNN
+	1    6400 1750
+	1    0    0    -1
+$EndComp
+Wire Wire Line
+	6400 1750 6400 1700
 Text Label 5250 7050 2    50   ~ 0
 TDI
@@
 Wire Wire Line
 	4950 5950 4950 6100
+$Comp
+L Device:Crystal Y?
+U 1 1 5C670581
+P 7350 1650
+F 0 "Y?" V 7350 1600 50  0000 L CNN
+F 1 "Crystal" V 7350 1750 50  0000 L CNN
+F 2 "" H 7350 1650 50  0001 C CNN
+F 3 "~" H 7350 1650 50  0001 C CNN
+	1    7350 1650
+	0    1    1    0
+$EndComp
+Wire Wire Line
+	6400 1400 7700 1400
+Wire Wire Line
+	7700 1700 7550 1700
+Wire Wire Line
+	7550 1700 7550 1800
+Wire Wire Line
+	7550 1800 7350 1800
+Wire Wire Line
+	7700 1600 7550 1600
+Wire Wire Line
+	7550 1600 7550 1500
+Wire Wire Line
+	7550 1500 7350 1500
+$Comp
+L Device:C_Small C?
+U 1 1 5C6C5E13
+P 7100 1500
+F 0 "C?" V 7150 1400 50  0000 C CNN
+F 1 "30p" V 7200 1500 50  0000 C CNN
+F 2 "Capacitor_SMD:C_0603_1608Metric_Pad1.05x0.95mm_HandSolder" H 7100 1500 50  0001 C CNN
+F 3 "~" H 7100 1500 50  0001 C CNN
+	1    7100 1500
+	0    1    1    0
+$EndComp
+$Comp
+L Device:C_Small C?
+U 1 1 5C6C5F00
+P 7100 1800
+F 0 "C?" V 7150 1700 50  0000 C CNN
+F 1 "30p" V 7200 1800 50  0000 C CNN
+F 2 "Capacitor_SMD:C_0603_1608Metric_Pad1.05x0.95mm_HandSolder" H 7100 1800 50  0001 C CNN
+F 3 "~" H 7100 1800 50  0001 C CNN
+	1    7100 1800
+	0    1    1    0
+$EndComp
+Wire Wire Line
+	7200 1500 7350 1500
+Connection ~ 7350 1500
+Wire Wire Line
+	7200 1800 7350 1800
+Connection ~ 7350 1800
+Wire Wire Line
+	7000 1500 6850 1500
+Wire Wire Line
+	6850 1500 6850 1650
+Wire Wire Line
+	6850 1800 7000 1800
+$Comp
+L power:GND #PWR?
+U 1 1 5C6E00F1
+P 6750 1650
+F 0 "#PWR?" H 6750 1400 50  0001 C CNN
+F 1 "GND" H 6755 1477 50  0000 C CNN
+F 2 "" H 6750 1650 50  0001 C CNN
+F 3 "" H 6750 1650 50  0001 C CNN
+	1    6750 1650
+	1    0    0    -1
+$EndComp
+Wire Wire Line
+	6750 1650 6850 1650
+Connection ~ 6850 1650
+Wire Wire Line
+	6850 1650 6850 1800
 $EndSCHEMATC

Commit message: Schematic almost complete
Parts:
- C1, C10, C11, C2, C3, C9: renamed from C?; footprint Capacitor_SMD:C_0603_1608Metric -> Capacitor_SMD:C_0603_1608Metric_Pad1.05x0.95mm_HandSolder
- C12, C13, C4, C5, C6: renamed from C?; footprint (none) -> Capacitor_SMD:C_0603_1608Metric_Pad1.05x0.95mm_HandSolder
- C15: renamed from C?; value C -> 0u1
- J1: renamed from J?; symbol Connectors:PJ-002A -> ParkingSystem-rescue:PJ-002A-Connectors
- J4: renamed from J?; footprint (none) -> Connector_PinSocket_2.54mm:PinSocket_1x04_P2.54mm_Horizontal
- LS1: renamed from LS?; footprint (none) -> Buzzers:AI-2437-TWT-R
- Q1, Q2, Q3, Q4, Q5: renamed from Q?; footprint (none) -> MOSFETS:SSM3K33R,LF; symbol MOSFETS:SSM3K333R,LF -> ParkingSystem-rescue:SSM3K333R,LF-MOSFETS
- R1, R3, R4, R5, R6, R7: renamed from R?; footprint (none) -> Resistor_SMD:R_0603_1608Metric_Pad1.05x0.95mm_HandSolder
- Y1: renamed from Y?; footprint (none) -> Crystal:Crystal_HC18-U_Vertical
- gave numbers to parts that had none: 16
Connections:
- wire segments 174 -> 176
- no-connect marks 0 -> 27

Commit message: PCB Layout started
Parts:
- C14: value 0.1u -> 0u1
- C6: value 4.7u -> 4u7
- J5: footprint Connector_Molex:Molex_Mega-Fit_76829-0108_2x04_P5.70mm_Vertical -> Connector_Molex:Molex_Micro-Fit_3.0_43045-0200_2x01_P3.00mm_Horizontal
- SW1: footprint (none) -> Button_Switch_SMD:SW_SPST_B3S-1000
Changed lines of the file:
@@
 Sheet 1 1
 Title "Parking Sensor Hardware"
-Date "2019-02-12"
-Rev ""
+Date "2019-02-15"
+Rev "v01"
 Comp ""
 Comment1 ""
@@
 P 4350 1350
 F 0 "C6" H 4465 1396 50  0000 L CNN
-F 1 "4.7u" H 4465 1305 50  0000 L CNN
+F 1 "4u7" H 4465 1305 50  0000 L CNN
 F 2 "Capacitor_SMD:C_0603_1608Metric_Pad1.05x0.95mm_HandSolder" H 4388 1200 50  0001 C CNN
 F 3 "~" H 4350 1350 50  0001 C CNN
@@
 F 0 "SW1" V 10404 4398 50  0000 L CNN
 F 1 "SW_Push" V 10495 4398 50  0000 L CNN
-F 2 "" H 10450 4450 50  0001 C CNN
+F 2 "Button_Switch_SMD:SW_SPST_B3S-1000" H 10450 4450 50  0001 C CNN
 F 3 "" H 10450 4450 50  0001 C CNN
 	1    10450 4250
@@
 P 10100 4250
 F 0 "C14" H 10215 4296 50  0000 L CNN
-F 1 "0.1u" H 10215 4205 50  0000 L CNN
+F 1 "0u1" H 10215 4205 50  0000 L CNN
 F 2 "Capacitor_SMD:C_0603_1608Metric_Pad1.05x0.95mm_HandSolder" H 10138 4100 50  0001 C CNN
 F 3 "~" H 10100 4250 50  0001 C CNN
@@
 F 0 "J5" H 2256 7625 50  0000 C CNN
 F 1 "0430450200" H 2256 7534 50  0000 C CNN
-F 2 "Connector_Molex:Molex_Mega-Fit_76829-0108_2x04_P5.70mm_Vertical" H 2200 7350 50  0001 C CNN
+F 2 "Connector_Molex:Molex_Micro-Fit_3.0_43045-0200_2x01_P3.00mm_Horizontal" H 2200 7350 50  0001 C CNN
 F 3 "" H 2200 7350 50  0001 C CNN
 	1    2200 7350

Commit message: Move for better placement
Connections:
- net +3V3: now also C15.1, U4.8 (VDD)
- net +5V: no longer C15.1, U4.8 (VDD)
- net INDICATOR: now also U3.45 (PB8)
- no-connect marks 27 -> 25
Changed lines of the file:
@@
 Wire Wire Line
 	10200 6200 10200 6100
-$Comp
-L power:+5V #PWR0135
-U 1 1 5C6484FC
-P 10200 5150
-F 0 "#PWR0135" H 10200 5000 50  0001 C CNN
-F 1 "+5V" H 10215 5323 50  0000 C CNN
-F 2 "" H 10200 5150 50  0001 C CNN
-F 3 "" H 10200 5150 50  0001 C CNN
-	1    10200 5150
-	1    0    0    -1
-$EndComp
 Wire Wire Line
 	10200 5150 10200 5300
@@
 F 3 "~" H 10950 5650 50  0001 C CNN
 	1    10950 5650
-	1    0    0    -1
-$EndComp
-$Comp
-L power:+5V #PWR0146
-U 1 1 5C66CFE9
-P 10950 5400
-F 0 "#PWR0146" H 10950 5250 50  0001 C CNN
-F 1 "+5V" H 10965 5573 50  0000 C CNN
-F 2 "" H 10950 5400 50  0001 C CNN
-F 3 "" H 10950 5400 50  0001 C CNN
-	1    10950 5400
 	1    0    0    -1
 $EndComp
@@
 NoConn ~ 7700 2700
 NoConn ~ 7700 2800
-NoConn ~ 7700 3150
 NoConn ~ 7700 3200
-NoConn ~ 7700 3100
 NoConn ~ 7700 3500
 NoConn ~ 7700 3600
@@
 	2750 6650 2350 6650
 NoConn ~ 10700 5700
+Text Label 7250 3100 0    50   ~ 0
+INDICATOR
+Wire Wire Line
+	7250 3100 7700 3100
+$Comp
+L power:+3V3 #PWR?
+U 1 1 5C6AC93A
+P 10200 5150
+F 0 "#PWR?" H 10200 5000 50  0001 C CNN
+F 1 "+3V3" H 10215 5323 50  0000 C CNN
+F 2 "" H 10200 5150 50  0001 C CNN
+F 3 "" H 10200 5150 50  0001 C CNN
+	1    10200 5150
+	1    0    0    -1
+$EndComp
+$Comp
+L power:+3V3 #PWR?
+U 1 1 5C6AC9DD
+P 10950 5400
+F 0 "#PWR?" H 10950 5250 50  0001 C CNN
+F 1 "+3V3" H 10965 5573 50  0000 C CNN
+F 2 "" H 10950 5400 50  0001 C CNN
+F 3 "" H 10950 5400 50  0001 C CNN
+	1    10950 5400
+	1    0    0    -1
+$EndComp
 $EndSCHEMATC

Commit message: Change MCU pin I/O lines and route
Parts:
- C1, C10, C11, C12, C13, C14, C15, C2, C3, C4, C5, C6, C9: symbol Device:C -> ParkingSystem-rescue:C-Device
- C7, C8: symbol Device:C_Small -> ParkingSystem-rescue:C_Small-Device
- D1: symbol Device:LED -> ParkingSystem-rescue:LED-Device
- J2: symbol Connectors:0430450400 -> ParkingSystem-rescue:0430450400-Connectors
- J3: symbol Connector:Conn_ARM_JTAG_SWD_10 -> ParkingSystem-rescue:Conn_ARM_JTAG_SWD_10-Connector
- J4: symbol Connector:Conn_01x04_Female -> ParkingSystem-rescue:Conn_01x04_Female-Connector
- J5: symbol Connectors:0430450200 -> ParkingSystem-rescue:0430450200-Connectors
- LS1: symbol Buzzers:AI-2437-TWT-R -> ParkingSystem-rescue:AI-2437-TWT-R-Buzzers
- R1, R10, R2, R3, R4, R5, R6, R7, R8, R9: symbol Device:R_US -> ParkingSystem-rescue:R_US-Device
- SW1: symbol Switch:SW_Push -> ParkingSystem-rescue:SW_Push-Switch
- U1: symbol Regulator_Switching:R-78E5.0-1.0 -> ParkingSystem-rescue:R-78E5.0-1.0-Regulator_Switching
- U2: symbol Regulator_Switching:R-783.3-0.5 -> ParkingSystem-rescue:R-783.3-0.5-Regulator_Switching
- U3: symbol MCU_ST_STM32F1:STM32F103C4Tx -> ParkingSystem-rescue:STM32F103C4Tx-MCU_ST_STM32F1
- U4: symbol Sensor_Temperature:DS1621S -> ParkingSystem-rescue:DS1621S-Sensor_Temperature
- Y1: symbol Device:Crystal -> ParkingSystem-rescue:Crystal-Device
Connections:
- net BLUE: now also U3.14 (PA4); no longer U3.21 (PB10)
- net BUZZER: now also U3.40 (PB4); no longer U3.14 (PA4)
- net GREEN: now also U3.15 (PA5); no longer U3.22 (PB11)
- net INDICATOR: now also U3.16 (PA6); no longer U3.45 (PB8)
- net RED: now also U3.13 (PA3); no longer U3.15 (PA5)
- net TRIG: now also U3.12 (PA2); no longer U3.10 (PA0)

Commit message: Add Mounting Holes
Parts:
- added H1, H2: MountingHole, MountingHole:MountingHole_4.3mm_M4_DIN965_Pad, symbol Mechanical:MountingHole
Changed lines of the file:
@@
 	9400 2900 9000 2900
 NoConn ~ 7700 3100
+$Comp
+L Mechanical:MountingHole H2
+U 1 1 5C69771C
+P 5600 7400
+F 0 "H2" H 5700 7446 50  0000 L CNN
+F 1 "MountingHole" H 5700 7355 50  0000 L CNN
+F 2 "MountingHole:MountingHole_4.3mm_M4_DIN965_Pad" H 5600 7400 50  0001 C CNN
+F 3 "~" H 5600 7400 50  0001 C CNN
+	1    5600 7400
+	1    0    0    -1
+$EndComp
+$Comp
+L Mechanical:MountingHole H1
+U 1 1 5C6978DE
+P 5600 7100
+F 0 "H1" H 5700 7146 50  0000 L CNN
+F 1 "MountingHole" H 5700 7055 50  0000 L CNN
+F 2 "MountingHole:MountingHole_4.3mm_M4_DIN965_Pad" H 5600 7100 50  0001 C CNN
+F 3 "~" H 5600 7100 50  0001 C CNN
+	1    5600 7100
+	1    0    0    -1
+$EndComp
 $EndSCHEMATC
